Commit message: Boxes and walls static

File: learning/urdf/wall.urdf (robot description, URDF)
Before this commit: robot wall, 2 links, 0 joints
Links:
- removed link world

File: learning/urdf/wall2.urdf (robot description, URDF)
Before this commit: robot wall, 2 links, 0 joints
Links:
- removed link world
- link my_wall: mass 100.0 -> 1.0

Commit message: Changed walls and order of actions

File: learning/urdf/wall.urdf (robot description, URDF)
Before this commit: robot wall, 1 links, 0 joints
Links:
- link my_wall: geometry collision box size=0.024171 5 0.05; visual box size=0.024171 5 0.05

File: learning/urdf/wall2.urdf (robot description, URDF)
Before this commit: robot wall, 1 links, 0 joints
Links:
- link my_wall: geometry collision box size=0.024171 11 0.05; visual box size=0.024171 11 0.05
