Commit message: Fixed image and object a bit bigger

File: learning/urdf/cylinder.urdf (robot description, URDF)
Before this commit: robot red_object, 1 links, 0 joints
Links:
- link my_object: geometry collision cylinder length=0.100067 radius=0.0150855; visual cylinder length=0.100067 radius=0.0150855

Commit message: Fixed decay, reward

File: learning/urdf/cylinder.urdf (robot description, URDF)
Before this commit: robot red_object, 1 links, 0 joints
Links:
- link my_object: geometry collision cylinder length=0.100067 radius=0.0100855; visual cylinder length=0.100067 radius=0.0100855

Commit message: Changed reward and cylinder size

File: learning/urdf/cylinder.urdf (robot description, URDF)
Before this commit: robot red_object, 1 links, 0 joints
Links:
- link my_object: geometry collision cylinder length=0.100067 radius=0.0120855; visual cylinder length=0.100067 radius=0.0120855
