Commit message: Controlled environment

File: ROS-master/crumb/crumb_description/urdf/sensors/kinect_crumb.urdf (copia).xacro (robot description, xacro)
@@ -3,5 +3,5 @@
   <xacro:include filename="$(find crumb_description)/urdf/turtlebot_gazebo_crumb.urdf.xacro"/>
   <xacro:include filename="$(find turtlebot_description)/urdf/turtlebot_properties.urdf.xacro"/>
-  <xacro:property name="kinect_cam_py" value="0.0"/>
+  <xacro:property name="kinect_cam_py" value="-0.0125"/>
   <!-- Parameterised in part by the values in turtlebot_properties.urdf.xacro -->
   <xacro:macro name="sensor_kinect_crumb" params="parent">
@@ -48,5 +48,5 @@
          (Hence, don't publish them additionally!) -->
 	<joint name="camera_depth_joint" type="fixed">
-	  <origin xyz="0 ${2 * 0.0125} 0" rpy="0 0 0" />
+	  <origin xyz="0 ${2 * -kinect_cam_py} 0" rpy="0 0 0" />
 	  <parent link="camera_rgb_frame" />
 	  <child link="camera_depth_frame" />

File: ROS-master/crumb/crumb_description/urdf/sensors/kinect_crumb_n.urdf (copia).xacro (robot description, xacro)
@@ -1,9 +1,9 @@
 <?xml version="1.0"?>
 <robot name="sensor_kinect" xmlns:xacro="http://ros.org/wiki/xacro">
-  <xacro:include filename="$(find crumb_description)/urdf/turtlebot_gazebo_crumb.urdf.xacro"/>
+  <xacro:include filename="$(find crumb_description)/urdf/turtlebot_gazebo_crumb_n.urdf.xacro"/>
   <xacro:include filename="$(find turtlebot_description)/urdf/turtlebot_properties.urdf.xacro"/>
-  <xacro:property name="kinect_cam_py" value="0.0"/>
+  <xacro:property name="kinect_cam_py" value="-0.0125"/>
   <!-- Parameterised in part by the values in turtlebot_properties.urdf.xacro -->
-  <xacro:macro name="sensor_kinect_crumb" params="parent">
+  <xacro:macro name="sensor_kinect_crumb_n" params="parent">
     <joint name="camera_rgb_joint" type="fixed">
       <origin xyz="${cam_px} ${kinect_cam_py} ${cam_pz}" rpy="${cam_or} ${cam_op} ${cam_oy}"/>
@@ -48,5 +48,5 @@
          (Hence, don't publish them additionally!) -->
 	<joint name="camera_depth_joint" type="fixed">
-	  <origin xyz="0 ${2 * 0.0125} 0" rpy="0 0 0" />
+	  <origin xyz="0 ${2 * -kinect_cam_py} 0" rpy="0 0 0" />
 	  <parent link="camera_rgb_frame" />
 	  <child link="camera_depth_frame" />
@@ -60,5 +60,5 @@
 	<link name="camera_depth_optical_frame"/>
 	<!-- Kinect sensor for simulation -->
-	<turtlebot_sim_3dsensor_crumb/>
+	<turtlebot_sim_3dsensor_crumb_n/>
   </xacro:macro>
 </robot>

File: ROS-master/crumb/crumb_description/urdf/sensors/kinect_crumb_n.urdf.xacro (robot description, xacro)
@@ -3,5 +3,5 @@
   <xacro:include filename="$(find crumb_description)/urdf/turtlebot_gazebo_crumb_n.urdf.xacro"/>
   <xacro:include filename="$(find turtlebot_description)/urdf/turtlebot_properties.urdf.xacro"/>
-  <xacro:property name="kinect_cam_py" value="-0.0125"/>
+  <xacro:property name="kinect_cam_py" value="0.0"/>
   <!-- Parameterised in part by the values in turtlebot_properties.urdf.xacro -->
   <xacro:macro name="sensor_kinect_crumb_n" params="parent">
@@ -48,5 +48,5 @@
          (Hence, don't publish them additionally!) -->
 	<joint name="camera_depth_joint" type="fixed">
-	  <origin xyz="0 ${2 * -kinect_cam_py} 0" rpy="0 0 0" />
+	  <origin xyz="0 ${2 * 0.0125} 0" rpy="0 0 0" />
 	  <parent link="camera_rgb_frame" />
 	  <child link="camera_depth_frame" />
